Commit message: URDF Update

File: urdf/ar2.urdf (robot description, URDF)
Before this commit: robot ar2, 7 links, 6 joints
Links:
- removed link base_link
- removed link link_1
- removed link link_2
- removed link link_3
- removed link link_4
- removed link link_5
- removed link link_6
- added link link0, mass 0.88065; collision mesh filename=meshes/link0.STL; visual mesh filename=meshes/link0.STL
- added link link1, mass 0.57738; collision mesh filename=meshes/link1.STL; visual mesh filename=meshes/link1.STL
- added link link2, mass 0.1787; collision mesh filename=meshes/link2.STL; visual mesh filename=meshes/link2.STL
- added link link3, mass 0.34936; collision mesh filename=meshes/link3.STL; visual mesh filename=meshes/link3.STL
- added link link4, mass 0.11562; collision mesh filename=meshes/link4.STL; visual mesh filename=meshes/link4.STL
- added link link5, mass 0.013863; collision mesh filename=meshes/link5.STL; visual mesh filename=meshes/link5.STL
- added link linkBase, mass 0.7102; collision mesh filename=meshes/linkBase.STL; visual mesh filename=meshes/linkBase.STL
Joints:
- removed joint joint_1
- removed joint joint_2
- removed joint joint_3
- removed joint joint_4
- removed joint joint_5
- removed joint joint_6
- added joint joint0: type continuous, parent linkBase, child link0, origin xyz=0 0 0.003445 rpy=3.1416 -1.0248E-21 -1.6736E-05, axis 0 0 1
- added joint joint1: type continuous, parent link0, child link1, origin xyz=0 0.064146 -0.16608 rpy=1.5708 0.5236 -1.5708, axis 0 0 1
- added joint joint2: type continuous, parent link1, child link2, origin xyz=0.1525 -0.26414 0 rpy=3.3431E-16 -1.4164E-16 -2.618, axis 0 0 -1
- added joint joint3: type continuous, parent link2, child link3, origin xyz=0 0 0.00675 rpy=1.5708 -1.2554 -1.5708, axis 0 0 -1
- added joint joint4: type continuous, parent link3, child link4, origin xyz=0 0 -0.22225 rpy=3.1416 0 -2.8262, axis -1 0 0
- added joint joint6: type continuous, parent link_4, child link_5, origin xyz=-0.000294 0 0.02117 rpy=0 0 3.1416, axis 0 0 -1
